Commit message: Update test_robot_new.urdf

File: test_robot.urdf (robot description, URDF)
Before this commit: robot test_robot, 5 links, 4 joints
Links:
- link BL_link: geometry collision mesh filename=package://test_robot_new/meshes/BL_link.STL; visual mesh filename=package://test_robot_new/meshes/BL_link.STL
- link FB_link: geometry collision mesh filename=package://test_robot_new/meshes/FB_link.STL; visual mesh filename=package://test_robot_new/meshes/FB_link.STL
- link FL_link: geometry collision mesh filename=package://test_robot_new/meshes/FL_link.STL; visual mesh filename=package://test_robot_new/meshes/FL_link.STL
- link FR_link: geometry collision mesh filename=package://test_robot_new/meshes/FR_link.STL; visual mesh filename=package://test_robot_new/meshes/FR_link.STL
- link base_link: geometry collision mesh filename=package://test_robot_new/meshes/base_link.STL; visual mesh filename=package://test_robot_new/meshes/base_link.STL

Commit message: Update test_robot_new.urdf

File: test_robot.urdf (robot description, URDF)
Before this commit: robot test_robot_new, 5 links, 4 joints
Links:
- added link dummy_link
Joints:
- added joint base_joint: type fixed, parent dummy_link, child base_link, origin xyz=0 0 0 rpy=0 0 0
